File: burstcart-via/burstcart-via/burstcart-via.kicad_pcb (KiCad board)
At the start: 2 copper layers, 56 x 91 mm, 24 parts, among them J1 IEC, J3 BURST, J4 PORTB, U1 27C512, U2 74LS74, U3 6522, U4 22V10, U5 74LS126

Commit message: finalized VIA board
Parts:
- JP3: footprint Jumper:SolderJumper-3_P1.3mm_Bridged12_Pad1.0x1.5mm_NumberLabels -> Jumper:SolderJumper-3_P1.3mm_Open_Pad1.0x1.5mm_NumberLabels
Changed lines of the file:
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@@
       (disableapertmacros false)
       (usegerberextensions true)
-      (usegerberattributes true)
-      (usegerberadvancedattributes true)
+      (usegerberattributes false)
+      (usegerberadvancedattributes false)
       (creategerberjobfile false)
       (svguseinch false)
@@
       (net 51 "/PHI0") (pinfunction "B") (pintype "passive"))
   )
-  (footprint "Jumper:SolderJumper-3_P1.3mm_Bridged12_Pad1.0x1.5mm_NumberLabels" (layer "B.Cu")
+  (footprint "Jumper:SolderJumper-3_P1.3mm_Open_Pad1.0x1.5mm_NumberLabels" (layer "B.Cu")
     (at 141.478 103.124 90)
-    (descr "SMD Solder Jumper, 1x1.5mm Pads, 0.3mm gap, pads 1-2 bridged with 1 copper strip, labeled with numbers")
-    (tags "net tie solder jumper bridged")
+    (descr "SMD Solder Jumper, 1x1.5mm Pads, 0.3mm gap, open, labeled with numbers")
+    (tags "solder jumper open")
     (property "Sheetfile" "burstcart-via.kicad_sch")
     (property "Sheetname" "")
     (attr exclude_from_pos_files)
-    (fp_text reference "JP3" (at 0 1.8 90) (layer "B.SilkS")
+    (fp_text reference "JP3" (at 0 1.8 270) (layer "B.SilkS")
       (effects (font (size 1 1) (thickness 0.15)) (justify mirror))
     )
-    (fp_text value "Jumper_3_Bridged12" (at 0 -1.9 90) (layer "B.Fab") hide
+    (fp_text value "Jumper_3_Bridged12" (at 0 -1.9 270) (layer "B.Fab")
       (effects (font (size 1 1) (thickness 0.15)) (justify mirror))
     )
-    (fp_text user "1" (at -2.6 0 90) (layer "B.SilkS")
+    (fp_text user "3" (at 2.6 0 270) (layer "B.SilkS")
       (effects (font (size 1 1) (thickness 0.15)) (justify mirror))
     )
-    (fp_text user "3" (at 2.6 0 90) (layer "B.SilkS")
+    (fp_text user "1" (at -2.6 0 270) (layer "B.SilkS")
       (effects (font (size 1 1) (thickness 0.15)) (justify mirror))
     )
-    (fp_poly (pts
-        (xy -0.9 0.3)
-        (xy -0.4 0.3)
-        (xy -0.4 -0.3)
-        (xy -0.9 -0.3)
-      ) (layer "B.Cu") (width 0) (fill solid))
+    (fp_line (start 2.05 -1) (end -2.05 -1) (layer "B.SilkS") (width 0.12))
     (fp_line (start 2.05 1) (end 2.05 -1) (layer "B.SilkS") (width 0.12))
     (fp_line (start -2.05 1) (end 2.05 1) (layer "B.SilkS") (width 0.12))
-    (fp_line (start 2.05 -1) (end -2.05 -1) (layer "B.SilkS") (width 0.12))
     (fp_line (start -2.05 -1) (end -2.05 1) (layer "B.SilkS") (width 0.12))
     (fp_line (start -2.3 1.25) (end -2.3 -1.25) (layer "B.CrtYd") (width 0.05))
+    (fp_line (start 2.3 -1.25) (end -2.3 -1.25) (layer "B.CrtYd") (width 0.05))
+    (fp_line (start -2.3 1.25) (end 2.3 1.25) (layer "B.CrtYd") (width 0.05))
     (fp_line (start 2.3 -1.25) (end 2.3 1.25) (layer "B.CrtYd") (width 0.05))
-    (fp_line (start -2.3 1.25) (end 2.3 1.25) (layer "B.CrtYd") (width 0.05))
-    (fp_line (start 2.3 -1.25) (end -2.3 -1.25) (layer "B.CrtYd") (width 0.05))
     (pad "1" smd rect (at -1.3 0 90) (size 1 1.5) (layers "B.Cu" "B.Mask")
       (net 21 "/PHI2") (pinfunction "A") (pintype "passive"))
