File: burstcart-via/burstcart-via/burstcart-via.kicad_sch (KiCad schematic)
At the start: 24 parts, among them J1 IEC, J3 BURST, J4 PORTB, U1 27C512, U2 74LS74, U3 6522, U4 22V10, U5 74LS126

Commit message: finalized VIA board
Parts:
- JP3: footprint Jumper:SolderJumper-3_P1.3mm_Bridged12_Pad1.0x1.5mm_NumberLabels -> Jumper:SolderJumper-3_P1.3mm_Open_Pad1.0x1.5mm_NumberLabels; symbol Jumper:Jumper_3_Bridged12 -> Jumper:Jumper_3_Open
Other:
- note added: "GAL CLOCK SELECTION (probably Phi0)"
- note removed: "GAL CLOCK SELECTION"
Changed lines of the file:
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@@
     (effects (font (size 1.27 1.27)) (justify left bottom))
   )
-  (text "GAL CLOCK\nSELECTION" (at 213.995 53.975 0)
+  (text "GAL CLOCK\nSELECTION\n(probably Phi0)" (at 213.995 53.975 0)
     (effects (font (size 1.27 1.27)) (justify left bottom))
   )
@@
     (pin "9")
   )
-  (symbol (lib_id "Jumper:Jumper_3_Bridged12") (at 217.17 63.5 90) (unit 1)
+  (symbol (lib_id "Jumper:Jumper_3_Open") (at 217.17 63.5 90) (unit 1)
     (in_bom yes) (on_board yes) (fields_autoplaced)
     (property "Reference" "JP3" (id 0) (at 214.63 63.4999 90)
@@
       (effects (font (size 1.27 1.27)) (justify left) hide)
     )
-    (property "Footprint" "Jumper:SolderJumper-3_P1.3mm_Bridged12_Pad1.0x1.5mm_NumberLabels" (id 2) (at 217.17 63.5 0)
+    (property "Footprint" "Jumper:SolderJumper-3_P1.3mm_Open_Pad1.0x1.5mm_NumberLabels" (id 2) (at 217.17 63.5 0)
       (effects (font (size 1.27 1.27)) hide)
     )
@@
     )
     (path "/3b511bdc-fdd2-476b-bc62-c0483bf6b3f0"
-      (reference "JP3") (unit 1) (value "Jumper_3_Bridged12") (footprint "Jumper:SolderJumper-3_P1.3mm_Bridged12_Pad1.0x1.5mm_NumberLabels")
+      (reference "JP3") (unit 1) (value "Jumper_3_Bridged12") (footprint "Jumper:SolderJumper-3_P1.3mm_Open_Pad1.0x1.5mm_NumberLabels")
     )
     (path "/6fdcac5e-1e7e-4702-b89b-f9333852c3de"
