File: burstcart-cia/burstcart.kicad_pcb (KiCad board)
At the start: 2 copper layers, 56 x 91 mm, 20 parts, among them J1 IEC, J2 IEC, J3 BURST, J4 PORTA, U1 27C512, U2 CD74HCT4520E, U3 6526 CIA, U4 22V10, U5 ATtiny85-20P

Commit message: finalized v1.1 cia board too
Parts:
- added JP4: Jumper_3_Bridged12, Jumper:SolderJumper-3_P1.3mm_Bridged2Bar12_Pad1.0x1.5mm_NumberLabels, B.Cu at (133.6, 125.0)
- JP3: value O:HW/C:SW -> C:HW/O:SW
Connections:
- U4 pad 23: /PHI2 -> Net-(JP4-Pad2)
- U5 pad 6: unconnected-(U5-Pad6) -> /MUX
Routing:
- net /PHI2: track 49.9 -> 114.1 mm
- net /D4: track 103.2 -> 67.6 mm, vias 4 -> 3
- net /MUX: track 52.2 -> 80.3 mm, vias 2 -> 3
- net /D1: track 78.0 -> 54.1 mm, vias 3 -> 2
- net /D3: track 84.9 -> 66.4 mm, vias 4 -> 3
- net /D0: track 58.9 -> 73.0 mm, vias 3 -> 4
- net Net-(JP4-Pad2): track 0.00 -> 13.0 mm
- net /PHI0: track 0.00 -> 12.0 mm, vias 0 -> 2
- net /D5: track 73.1 -> 62.6 mm, vias 1 -> 2
- net /A2: track 63.5 -> 73.9 mm, vias 4 -> 3
- net /~{FLAG}: track 79.1 -> 68.7 mm, vias 1 -> 0
- net GND: track 246.8 -> 255.4 mm, vias 7 -> 8
- net /D6: track 68.1 -> 59.7 mm
- net /A4: track 32.2 -> 40.6 mm, vias 0 -> 2
- net /~{ROMCS}: track 67.9 -> 59.7 mm, vias 2 -> 3
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Other:
- board text added: "BurstCart+4 v1.1 Maciej Witkowiak, V 2025 <ytm@elysium.pl>"
- board text added: "Ph2 | GAL | Ph0"
- board text added: "Reset | out | GND"
- board text added: "Slow | CIA | Ph2"
- board text removed: "3-2: SLOW 2-1: FAST"
- board text removed: "BurstCart+4 v1.1 Maciej <ytm@elysium.pl> Witkowiak, V 2025"
