File: burstcart-cia/burstcart.kicad_sch (KiCad schematic)
At the start: 20 parts, among them J1 IEC, J2 IEC, J3 BURST, J4 PORTA, U1 27C512, U2 CD74HCT4520E, U3 6526 CIA, U4 22V10, U5 ATtiny85-20P

Commit message: finalized v1.1 cia board too
Parts:
- added JP4: Jumper_3_Bridged12, Jumper:SolderJumper-3_P1.3mm_Bridged2Bar12_Pad1.0x1.5mm_NumberLabels, symbol Jumper:Jumper_3_Bridged12
Connections:
- net MUX: now also U5.6 (PB1)
- net PHI0: now also JP4.1 (A)
- net PHI2: now also JP4.3 (B); no longer U4.23 (I12)
- new net: JP4.2 (C), U4.23 (I12)
- no-connect marks 21 -> 19
Other:
- note added: "PHI2 IS NECESSARY FOR ADDRESS DECODING BECAUSE ADDRESSES ARE VALID ON ITS RISING EDGE MW: It seems reliable option is Phi0 for GAL and Phi2 for CIA"
- note removed: "PHI2 IS NECESSARY FOR ADDRESS DECODING BECAUSE ADDRESSES ARE VALID ON ITS RISING EDGE"
Changed lines of the file:
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@@
   (title_block
     (title "BurstCart+4")
-    (date "2025-05-01")
+    (date "2025-05-07")
     (rev "1.1")
     (company "YTM Enterprises")
@@
   (no_connect (at 128.27 59.055))
   (no_connect (at 148.59 27.305))
-  (no_connect (at 235.585 95.25))
   (no_connect (at 27.305 33.655))
   (no_connect (at 235.585 97.79))
   (no_connect (at 75.565 64.135))
   (no_connect (at 128.27 56.515))
-  (no_connect (at 27.305 79.375))
   (no_connect (at 75.565 36.195))
   (no_connect (at 75.565 66.675))
@@
     (stroke (width 0) (type default) (color 0 0 0 0))
   )
+  (wire (pts (xy 234.95 67.31) (xy 244.475 67.31))
+    (stroke (width 0) (type default) (color 0 0 0 0))
+  )
   (wire (pts (xy 152.4 62.23) (xy 161.925 62.23))
     (stroke (width 0) (type default) (color 0 0 0 0))
@@
     (effects (font (size 1.27 1.27)) (justify left bottom))
   )
-  (text "closed = SW delay clock\nopen = HW prescaler clock" (at 237.49 98.425 0)
+  (text "closed = SW delay clock\nopen = HW prescaler clock" (at 249.555 97.79 0)
     (effects (font (size 1.27 1.27)) (justify left bottom))
   )
@@
     (effects (font (size 1.27 1.27)) (justify left bottom))
   )
-  (text "PHI2 IS NECESSARY FOR ADDRESS\nDECODING BECAUSE ADDRESSES\nARE VALID ON ITS RISING EDGE"
-    (at 205.74 59.055 0)
+  (text "PHI2 IS NECESSARY FOR ADDRESS\nDECODING BECAUSE ADDRESSES\nARE VALID ON ITS RISING EDGE\n\nMW: It seems reliable option is\nPhi0 for GAL and Phi2 for CIA"
+    (at 189.865 69.85 0)
     (effects (font (size 1.27 1.27)) (justify left bottom))
   )
@@
     (effects (font (size 1.27 1.27)) (justify left bottom))
   )
+  (label "PHI0" (at 231.14 73.66 180)
+    (effects (font (size 0.889 0.889)) (justify right bottom))
+  )
   (label "D2" (at 102.235 122.555 0)
     (effects (font (size 1.016 1.016)) (justify left bottom))
@@
   )
   (label "TOD" (at 242.57 92.71 0)
-    (effects (font (size 1.27 1.27)) (justify left bottom))
+    (effects (font (size 1.016 1.016)) (justify left bottom))
   )
   (label "reset" (at 269.875 52.07 0)
@@
     (effects (font (size 1.016 1.016)) (justify left bottom))
   )
+  (label "MUX" (at 235.585 95.25 0)
+    (effects (font (size 1.016 1.016)) (justify left bottom))
+  )
   (label "GND" (at 75.565 28.575 0)
     (effects (font (size 0.889 0.889)) (justify left bottom))
@@
     (effects (font (size 1.27 1.27)) (justify left bottom))
   )
-  (label "PHI2" (at 244.475 67.31 180)
-    (effects (font (size 1.27 1.27)) (justify right bottom))
+  (label "PHI2" (at 231.14 60.96 180)
+    (effects (font (size 0.889 0.889)) (justify right bottom))
   )
   (label "D4" (at 75.565 48.895 0)
@@
       (effects (font (size 1.27 1.27)) hide)
     )
-    (pin "1")
-    (pin "2")
-    (pin "3")
-    (pin "4")
-    (pin "5")
-    (pin "6")
-    (pin "7")
     (pin "10")
     (pin "11")
@@
     (pin "15")
     (pin "9")
-    (pin "16")
-    (pin "8")
   )
   (symbol (lib_id "4xxx:4520") (at 152.4 49.53 0) (unit 3)
@@
       (effects (font (size 1.27 1.27)) hide)
     )
-    (pin "1")
-    (pin "2")
-    (pin "3")
-    (pin "4")
-    (pin "5")
-    (pin "6")
-    (pin "7")
-    (pin "10")
-    (pin "11")
-    (pin "12")
-    (pin "13")
-    (pin "14")
-    (pin "15")
-    (pin "9")
     (pin "16")
     (pin "8")
@@
     (pin "6")
     (pin "7")
-    (pin "10")
-    (pin "11")
-    (pin "12")
-    (pin "13")
-    (pin "14")
-    (pin "15")
-    (pin "9")
-    (pin "16")
-    (pin "8")
   )
   (symbol (lib_id "Device:C") (at 255.27 147.955 0) (unit 1)
@@
     (pin "8")
     (pin "9")
-    (pin "1")
-    (pin "20")
   )
   (symbol (lib_id "MCU_Microchip_ATtiny:ATtiny85-20P") (at 220.345 100.33 0) (unit 1)
@@
       (effects (font (size 1.27 1.27)) hide)
     )
-    (pin "10")
-    (pin "11")
-    (pin "12")
-    (pin "13")
-    (pin "14")
-    (pin "15")
-    (pin "16")
-    (pin "17")
-    (pin "18")
-    (pin "19")
-    (pin "2")
-    (pin "21")
-    (pin "22")
-    (pin "23")
-    (pin "24")
-    (pin "25")
-    (pin "26")
-    (pin "27")
-    (pin "28")
-    (pin "29")
-    (pin "3")
-    (pin "30")
-    (pin "31")
-    (pin "32")
-    (pin "33")
-    (pin "34")
-    (pin "35")
-    (pin "36")
-    (pin "37")
-    (pin "38")
-    (pin "39")
-    (pin "4")
-    (pin "40")
-    (pin "5")
-    (pin "6")
-    (pin "7")
-    (pin "8")
-    (pin "9")
     (pin "1")
     (pin "20")
@@
     (pin "8")
     (pin "9")
-    (pin "12")
-    (pin "24")
   )
   (symbol (lib_id "power:GND") (at 220.345 115.57 0) (unit 1)
@@
       (effects (font (size 1.27 1.27)) hide)
     )
-    (pin "1")
-    (pin "10")
-    (pin "11")
-    (pin "13")
-    (pin "14")
-    (pin "15")
-    (pin "16")
-    (pin "17")
-    (pin "18")
-    (pin "19")
-    (pin "2")
-    (pin "20")
-    (pin "21")
-    (pin "22")
-    (pin "23")
-    (pin "3")
-    (pin "4")
-    (pin "5")
-    (pin "6")
-    (pin "7")
-    (pin "8")
-    (pin "9")
     (pin "12")
     (pin "24")
+  )
+  (symbol (lib_id "Jumper:Jumper_3_Bridged12") (at 231.14 67.31 90) (unit 1)
+    (in_bom yes) (on_board yes) (fields_autoplaced)
+    (property "Reference" "JP4" (id 0) (at 229.235 67.3099 90)
+      (effects (font (size 1.27 1.27)) (justify left))
+    )
+    (property "Value" "Jumper_3_Bridged12" (id 1) (at 228.6 68.5799 90)
+      (effects (font (size 1.27 1.27)) (justify left) hide)
+    )
+    (property "Footprint" "Jumper:SolderJumper-3_P1.3mm_Bridged2Bar12_Pad1.0x1.5mm_NumberLabels" (id 2) (at 231.14 67.31 0)
+      (effects (font (size 1.27 1.27)) hide)
+    )
+    (property "Datasheet" "~" (id 3) (at 231.14 67.31 0)
+      (effects (font (size 1.27 1.27)) hide)
+    )
+    (pin "1")
+    (pin "2")
+    (pin "3")
   )
   (symbol (lib_id "Jumper:SolderJumper_2_Open") (at 246.38 100.33 0) (unit 1)
@@
       (reference "JP3") (unit 1) (value "HW/SW") (footprint "Jumper:SolderJumper-2_P1.3mm_Open_Pad1.0x1.5mm")
     )
+    (path "/dc121f4e-0673-4834-a909-ead2af2c069f"
+      (reference "JP4") (unit 1) (value "Jumper_3_Bridged12") (footprint "Jumper:SolderJumper-3_P1.3mm_Bridged2Bar12_Pad1.0x1.5mm_NumberLabels")
+    )
     (path "/2a6f72c5-6e17-4a4c-b906-94df7dcb13bf"
