File: burstcart-via/kicad/burstcart-via.kicad_sch (KiCad schematic)
At the start: 24 parts, among them J1 IEC, J3 BURST, J4 PORTB, U1 27C512, U2 74LS74, U3 6522, U4 22V10, U5 74LS126

Commit message: corrected JP4 to connect to Phi0 by default, corrected silkscreen texts ; updated to KiCad9
Parts:
- JP3: footprint Jumper:SolderJumper-3_P1.3mm_Open_Pad1.0x1.5mm_NumberLabels -> Jumper:SolderJumper-3_P1.3mm_Bridged12_Pad1.0x1.5mm_NumberLabels; symbol Jumper:Jumper_3_Open -> Jumper:Jumper_3_Bridged12; now left out of the parts list
Connections:
- net PHI0: now also JP3.1 (A); no longer JP3.3 (B)
- net PHI2: now also JP3.3 (B); no longer JP3.1 (A)
Other:
- note added: "1-2: W65C22S"
- note added: "3-2: All other 6522 models"
- note added: "GAL CLOCK SELECTION"
- note added: "PHIx IS NECESSARY FOR ADDRESS DECODING BECAUSE ADDRESSES ARE VALID ON ITS RISING EDGE"
- note added: "VIA#1 in 1541 to VIA in +4 39. ~{CA2} - 40. ~{CA1} / ~{FLAG} in CIA 2. PA0 - PA0 3. PA1 - PA1 4. PA2 - PA2 5. PA3 - PA3 6. PA4 - PA4 7. PA5 - PA5 8. PA6 - PA6 9. PA7 - PA7 18. ~{CB1} - 39. ~{CA2} / ~{PC} in CIA"
- note removed: "All other 6522 models"
- note removed: "GAL CLOCK SELECTION (probably Phi0)"
- note removed: "PHI2 IS NECESSARY FOR ADDRESS DECODING BECAUSE ADDRESSES ARE VALID ON ITS RISING EDGE"
- note removed: "VIA#1 in 1541 to CIA#2 39, ~{CA2} - ~{FLAG} 2, PA0 - PB0 3, PA1 - PB1 4, PA2 - PB2 5, PA3 - PB3 6, PA4 - PB4 7, PA5 - PB5 8, PA6 - PB6 9, PA7 - PB7 18, CB1 - ~{PC}"
- note removed: "W65C22S"
